File: elektroonika/x-jalad rev2.sch (EAGLE design)
At the start: 53 parts, among them Q1 FC-12M

Commit message: eagle files init
Parts:
- removed VREF1, VREF2, VREF3, VREF4: (no value), wirepad:3,17/1,3
- added C2, C6: 100nF, eagle-ltspice:CC0402
- added C7: 4.7uF, rcl:C-EUC0603
- added LED4: (no value), led:LEDLD260
- added R18: 1k, rcl:R-EU_R0603
- added R20: 1k, eagle-ltspice:RR0402
- added U$11: MOLEX-530470210, pwr_connector:MOLEX-530470210
- C1, C4: device eagle-ltspice:CC0402 -> rcl:C-EUC0603
- C5: value 4.7 uF -> (none)
- JP1: device pinhead:PINHD-1X2/90 -> SparkFun:PINHD-2X3
- R16, R17, R4, R5, R6, R7: device eagle-ltspice:RR0402 -> rcl:R-EU_R0603
- U$10, U$9: value MOLEX-530470210 -> TE_CONNECTIVITY_2-1445055-2; device pwr_connector:MOLEX-530470210 -> Pressure_sensor_connector:TE_CONNECTIVITY_2-1445055-2
Connections:
- net NRST1 renamed HWB
- removed net TRGGR: 2CH_IDEAL_DIODES.ENBA, U$6.RST
- new net LED4: R18.2, U$2.PB7(OC0A/OC1C/RTS)
- new net N$10: 2CH_IDEAL_DIODES.INA, C7.1, R20.2
- new net N$7: LED4.A, R18.1
- new net N$8: U$8.3, U$8.6
- new net N$9: 2CH_IDEAL_DIODES.ENBA, C6.2, U$6.RST
- net +3V3: now also R20.1, U$8.2; no longer 2CH_IDEAL_DIODES.INA, C1.2, RTC.VBAT, U$4.VBAT, U$8.5
- net +5V: now also U$2.VBUS
- net GND: now also C2.2, C6.1, C7.2, JP1.6, LED4.C, U$11.1; no longer JP1.1, VREF2.P, VREF4.P
- net LED0: now also R6.2; no longer R7.2
- net LED1: now also R5.2; no longer R6.2
- net LED2: now also R4.2; no longer R5.2
- net LED3: now also R7.2; no longer R4.2
- net MISO: now also JP1.3
- net MOSI: now also JP1.5
- net N$2: now also C1.2, RTC.VBAT, U$11.2, U$4.VBAT, U$4.VBAT2, U$8.5; no longer JP1.2, U$8.2
- net NRST: now also JP1.4
- net S0_ADC: no longer VREF1.P
- net S1_ADC: no longer VREF3.P
- net SCK: now also JP1.1
- net VCC: now also C2.1, JP1.2; no longer U$2.VBUS
- net VCC/2: now also LDO.EN
Other:
- note removed: "Peab leidma õiget konnektorit"
- moved on the sheet: C3, C4, R11, R14, R16, R17, U$10, U$6, U$9
